File: pcb/switch42.kicad_pcb (KiCad board)
At the start: 2 copper layers, 91 x 55 mm, 25 parts, among them SW1 SW_PUSH, SW10 SW_PUSH, SW2 SW_PUSH, SW3 SW_PUSH, SW4 SW_PUSH, SW5 SW_PUSH, SW6 SW_PUSH, SW8 SW_PUSH, SW9 SW_PUSH, U1 ProMicro

Commit message: Update texts
Other:
- board text added: "1"
- board text added: "1. Flash the firmware on a ProMicro available here: https://github.com/zk-phi/qmk_firmware $ sh util/<your_OS>_install.sh $ make handwired/ddm9:default:avrdude 2. Solder x9 SK6812mini LEDs (Optional) * connected in serial 1 > 2 > 3 > … 3. Solder x9 Kailh Choc switches * cut pins marked with “X” 4. Plug ProMicro in with “Conthrough”s"
- board text added: "2"
- board text added: "3"
- board text added: "4"
- board text added: "5"
- board text added: "6"
- board text added: "64 and 13 me ! (I=“ai”, 0=zero) SFVIIDB6ciBMMXINCmdjbiAwY3 QgVDQ0DQp+RiEgcjJhIFpsMQ=="
- board text added: "7"
- board text added: "8"
- board text added: "9"
- board text added: "DDM Meishi Keypad rev.2"
- board text removed: "1. Flash the firmware on a ProMicro available here: https://github.com/zk-phi/qmk_firmware $ sh util/<your_OS>_install.sh $ make handwired/ddm9:default:avrdude 2. Solder x9 SK6812mini LEDs (Optional) * connected in serial D1 > D2 > … 3. Solder x9 Kailh Choc switches * cut pins marked with “X” 4. Plug ProMicro in with “Conthrough”s"
- board text removed: "D1"
- board text removed: "D2"
- board text removed: "D3"
- board text removed: "D4"
- board text removed: "D5"
- board text removed: "D6"
- board text removed: "D7"
- board text removed: "D8"
- board text removed: "D9"
- board text removed: "“64” and “13” me ! (I = “ai”) SFVIIDB6ciBMMXINCmdjbiAwY3 QgVDQ0DQp+RiEgcjJhIFpsMQ=="
Changed lines of the file:
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@@
   (general
     (thickness 1.6)
-    (drawings 79)
+    (drawings 80)
     (tracks 112)
     (zones 0)
@@
     )
   )
+  (gr_text "DDM Meishi Keypad rev.2" (at 127 103.5) (layer F.Cu)
+    (effects (font (size 1 1) (thickness 0.2)))
+  )
   (gr_text X (at 115 56.75) (layer B.SilkS)
     (effects (font (size 1 1) (thickness 0.2)) (justify mirror))
@@
     (effects (font (size 1 1) (thickness 0.2)) (justify mirror))
   )
-  (gr_text D9 (at 134.75 99) (layer B.SilkS)
+  (gr_text 9 (at 134.25 99) (layer B.SilkS)
     (effects (font (size 1 1) (thickness 0.2)) (justify mirror))
   )
-  (gr_text D8 (at 116.75 99) (layer B.SilkS)
+  (gr_text 8 (at 116.25 99) (layer B.SilkS)
     (effects (font (size 1 1) (thickness 0.2)) (justify mirror))
   )
-  (gr_text D7 (at 98.75 99) (layer B.SilkS)
+  (gr_text 7 (at 98.25 99) (layer B.SilkS)
     (effects (font (size 1 1) (thickness 0.2)) (justify mirror))
   )
-  (gr_text D6 (at 134.75 82) (layer B.SilkS)
+  (gr_text 6 (at 134.25 82) (layer B.SilkS)
     (effects (font (size 1 1) (thickness 0.2)) (justify mirror))
   )
-  (gr_text D5 (at 116.75 82) (layer B.SilkS)
+  (gr_text 5 (at 116.25 82) (layer B.SilkS)
     (effects (font (size 1 1) (thickness 0.2)) (justify mirror))
   )
-  (gr_text D4 (at 98.75 82) (layer B.SilkS)
+  (gr_text 4 (at 98.25 82) (layer B.SilkS)
     (effects (font (size 1 1) (thickness 0.2)) (justify mirror))
   )
-  (gr_text D3 (at 134.75 65) (layer B.SilkS)
+  (gr_text 3 (at 134.25 65) (layer B.SilkS)
     (effects (font (size 1 1) (thickness 0.2)) (justify mirror))
   )
-  (gr_text D2 (at 116.75 65) (layer B.SilkS)
+  (gr_text 2 (at 116.25 65) (layer B.SilkS)
     (effects (font (size 1 1) (thickness 0.2)) (justify mirror))
   )
-  (gr_text D1 (at 98.75 65) (layer B.SilkS)
+  (gr_text 1 (at 98.25 65) (layer B.SilkS)
     (effects (font (size 1 1) (thickness 0.2)) (justify mirror))
   )
@@
     (effects (font (size 1 1) (thickness 0.2)))
   )
-  (gr_text "Build your keypad !" (at 66.5 59.75) (layer B.SilkS)
+  (gr_text "Build your keypad !" (at 66.5 60.5) (layer B.SilkS)
     (effects (font (size 1 0.9) (thickness 0.2)) (justify mirror))
   )
-  (gr_text "“64” and “13” me ! (I = “ai”)\nSFVIIDB6ciBMMXINCmdjbiAwY3\nQgVDQ0DQp+RiEgcjJhIFpsMQ==" (at 81.25 100.75) (layer B.Cu)
+  (gr_text "64 and 13 me ! (I=“ai”, 0=zero)\nSFVIIDB6ciBMMXINCmdjbiAwY3\nQgVDQ0DQp+RiEgcjJhIFpsMQ==" (at 81.25 100.75) (layer B.Cu)
     (effects (font (size 0.9 0.9) (thickness 0.2)) (justify left mirror))
   )
-  (gr_text https://github.com/zk-phi/ddm9 (at 66.75 95.25) (layer B.SilkS)
+  (gr_text https://github.com/zk-phi/ddm9 (at 66.75 94.5) (layer B.SilkS)
     (effects (font (size 1 0.9) (thickness 0.2)) (justify mirror))
   )
@@
   )
   (gr_line (start 136.5 50) (end 136.5 105) (layer Cmts.User) (width 0.6))
-  (gr_text "1. Flash the firmware on a ProMicro\n\navailable here:\nhttps://github.com/zk-phi/qmk_firmware\n\n$ sh util/<your_OS>_install.sh\n$ make handwired/ddm9:default:avrdude\n\n2. Solder x9 SK6812mini LEDs (Optional)\n   * connected in serial D1 > D2 > …\n\n3. Solder x9 Kailh Choc switches\n   * cut pins marked with “X”\n\n4. Plug ProMicro in with “Conthrough”s" (at 81.25 77.5) (layer B.SilkS)
+  (gr_text "1. Flash the firmware on a ProMicro\n\navailable here:\nhttps://github.com/zk-phi/qmk_firmware\n\n$ sh util/<your_OS>_install.sh\n$ make handwired/ddm9:default:avrdude\n\n2. Solder x9 SK6812mini LEDs (Optional)\n   * connected in serial 1 > 2 > 3 > …\n\n3. Solder x9 Kailh Choc switches\n   * cut pins marked with “X”\n\n4. Plug ProMicro in with “Conthrough”s" (at 81.25 77.5) (layer B.SilkS)
     (effects (font (size 1 0.9) (thickness 0.2)) (justify left mirror))
   )

Commit message: Update texts
Other:
- board text added: "64 and 13 me ! (I=“ai”, 0=zero) WnJ+IFQwZyBMMEgNCmwyRiA0Y2 MgMXpVDQoxYSEgNHRuIHJySA=="
- board text removed: "64 and 13 me ! (I=“ai”, 0=zero) SFVIIDB6ciBMMXINCmdjbiAwY3 QgVDQ0DQp+RiEgcjJhIFpsMQ=="
Changed lines of the file:
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@@
     (effects (font (size 1 0.9) (thickness 0.2)) (justify mirror))
   )
-  (gr_text "64 and 13 me ! (I=“ai”, 0=zero)\nSFVIIDB6ciBMMXINCmdjbiAwY3\nQgVDQ0DQp+RiEgcjJhIFpsMQ==" (at 81.25 100.75) (layer B.Cu)
+  (gr_text "64 and 13 me ! (I=“ai”, 0=zero)\nWnJ+IFQwZyBMMEgNCmwyRiA0Y2\nMgMXpVDQoxYSEgNHRuIHJySA==" (at 81.25 100.75) (layer B.Cu)
     (effects (font (size 0.9 0.9) (thickness 0.2)) (justify left mirror))
   )

Commit message: Update texts
Other:
- board text added: "64 and 13 me ! (I=“ai”, 0=zero) WnJ+IFQwZyBMMEgNCmwyRiA0Y2 MgMXpVDQoxYSEgNHQ0IHJySA=="
- board text removed: "64 and 13 me ! (I=“ai”, 0=zero) WnJ+IFQwZyBMMEgNCmwyRiA0Y2 MgMXpVDQoxYSEgNHRuIHJySA=="
Changed lines of the file:
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@@
     (effects (font (size 1 0.9) (thickness 0.2)) (justify mirror))
   )
-  (gr_text "64 and 13 me ! (I=“ai”, 0=zero)\nWnJ+IFQwZyBMMEgNCmwyRiA0Y2\nMgMXpVDQoxYSEgNHRuIHJySA==" (at 81.25 100.75) (layer B.Cu)
+  (gr_text "64 and 13 me ! (I=“ai”, 0=zero)\nWnJ+IFQwZyBMMEgNCmwyRiA0Y2\nMgMXpVDQoxYSEgNHQ0IHJySA==" (at 81.25 100.75) (layer B.Cu)
     (effects (font (size 0.9 0.9) (thickness 0.2)) (justify left mirror))
   )

Commit message: Fix texts
Other:
- board text added: "64 and 13 me! (I=“ai”,0=zero) WnJ+IFQwZyBMMEgNCmwyRiA0Y2 MgMXpVDQoxYSEgNHQ0IHJySA=="
- board text added: "Build your keypad!"
- board text added: "DDM9 Meishi Keypad rev.2"
- board text removed: "64 and 13 me ! (I=“ai”, 0=zero) WnJ+IFQwZyBMMEgNCmwyRiA0Y2 MgMXpVDQoxYSEgNHQ0IHJySA=="
- board text removed: "Build your keypad !"
- board text removed: "DDM Meishi Keypad rev.2"
Changed lines of the file:
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@@
     )
   )
-  (gr_text "DDM Meishi Keypad rev.2" (at 127 103.5) (layer F.Cu)
+  (gr_text "DDM9 Meishi Keypad rev.2" (at 126.5 103.5) (layer F.Cu)
     (effects (font (size 1 1) (thickness 0.2)))
   )
@@
     (effects (font (size 1 1) (thickness 0.2)))
   )
-  (gr_text "Build your keypad !" (at 66.5 60.5) (layer B.SilkS)
+  (gr_text "Build your keypad!" (at 66.5 60.5) (layer B.SilkS)
     (effects (font (size 1 0.9) (thickness 0.2)) (justify mirror))
   )
-  (gr_text "64 and 13 me ! (I=“ai”, 0=zero)\nWnJ+IFQwZyBMMEgNCmwyRiA0Y2\nMgMXpVDQoxYSEgNHQ0IHJySA==" (at 81.25 100.75) (layer B.Cu)
+  (gr_text "64 and 13 me!  (I=“ai”,0=zero)\nWnJ+IFQwZyBMMEgNCmwyRiA0Y2\nMgMXpVDQoxYSEgNHQ0IHJySA==" (at 81.25 100.75) (layer B.Cu)
     (effects (font (size 0.9 0.9) (thickness 0.2)) (justify left mirror))
   )
