File: pcb/switch42.kicad_pcb (KiCad board)
At the start: 2 copper layers, 91 x 55 mm, 25 parts, among them SW1 SW_PUSH, SW10 SW_PUSH, SW2 SW_PUSH, SW3 SW_PUSH, SW4 SW_PUSH, SW5 SW_PUSH, SW6 SW_PUSH, SW8 SW_PUSH, SW9 SW_PUSH, U1 ProMicro

Commit message: Update texts
Other:
- board text added: "The key’s 0xD, the base’s 0x40. WnJ+fFRiZ3xMYmgKbDJGfDRj Y3wxeiMKMWEhfDRUNHxyckgK"
- board text removed: "64 and 13 me! (I=“ai”,0=zero) WnJ+IFQwZyBMMEgNCmwyRiA0Y2 MgMXpVDQoxYSEgNHQ0IHJySA=="
Changed lines of the file:
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@@
   (general
     (thickness 1.6)
-    (drawings 80)
+    (drawings 81)
     (tracks 112)
     (zones 0)
@@
     )
   )
+  (gr_line (start 73.5 61.25) (end 59.5 61.25) (layer B.SilkS) (width 0.2))
   (gr_text "DDM9 Meishi Keypad rev.2" (at 126.5 103.5) (layer F.Cu)
     (effects (font (size 1 1) (thickness 0.2)))
@@
   )
   (gr_text "Build your keypad!" (at 66.5 60.5) (layer B.SilkS)
-    (effects (font (size 1 0.9) (thickness 0.2)) (justify mirror))
-  )
-  (gr_text "64 and 13 me!  (I=“ai”,0=zero)\nWnJ+IFQwZyBMMEgNCmwyRiA0Y2\nMgMXpVDQoxYSEgNHQ0IHJySA==" (at 81.25 100.75) (layer B.Cu)
-    (effects (font (size 0.9 0.9) (thickness 0.2)) (justify left mirror))
+    (effects (font (size 1 1) (thickness 0.2)) (justify mirror))
+  )
+  (gr_text "The key’s 0xD, the base’s 0x40.\nWnJ+fFRiZ3xMYmgKbDJGfDRj\nY3wxeiMKMWEhfDRUNHxyckgK" (at 81.25 100.75) (layer B.Cu)
+    (effects (font (size 1 1) (thickness 0.2)) (justify left mirror))
   )
   (gr_text https://github.com/zk-phi/ddm9 (at 66.75 94.5) (layer B.SilkS)
-    (effects (font (size 1 0.9) (thickness 0.2)) (justify mirror))
+    (effects (font (size 1 1) (thickness 0.2)) (justify mirror))
   )
   (gr_text + (at 107.75 83) (layer B.SilkS)

Commit message: Update texts
Other:
- board text added: "Based on 0x40, the key is 0xD. WnJ+LFRiZyxMYmgKbDJGLG5 jYywxeiMKMWEhLDRUbixyckgK"
- board text removed: "The key’s 0xD, the base’s 0x40. WnJ+fFRiZ3xMYmgKbDJGfDRj Y3wxeiMKMWEhfDRUNHxyckgK"
Changed lines of the file:
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@@
     (effects (font (size 1 1) (thickness 0.2)) (justify mirror))
   )
-  (gr_text "The key’s 0xD, the base’s 0x40.\nWnJ+fFRiZ3xMYmgKbDJGfDRj\nY3wxeiMKMWEhfDRUNHxyckgK" (at 81.25 100.75) (layer B.Cu)
+  (gr_text "Based on 0x40, the key is 0xD.\nWnJ+LFRiZyxMYmgKbDJGLG5\njYywxeiMKMWEhLDRUbixyckgK" (at 81.25 100.75) (layer B.Cu)
     (effects (font (size 1 1) (thickness 0.2)) (justify left mirror))
   )

Commit message: Replace footprints
Parts:
- G***: footprint paripi:Untitled -> paripi:Untitled5
- G***: footprint paripi:Untitled2 -> paripi:Untitled6
